Commit message: modified:   README.md 	modified:   images/key_ctrl.png 	modified:   images/roarm_driver.py.png 	new file:   images/rviz_hand_tcp.png 	deleted:    images/rviz_link4.png 	modified:   src/roarm_main/moveit_servo/config/roarm_simulated_config.yaml 	modified:   src/roarm_main/moveit_servo/include/moveit_servo/servo_parameters.h 	modified:   src/roarm_main/moveit_servo/launch/demo.launch.py 	modified:   src/roarm_main/moveit_servo/src/servo_calcs.cpp 	modified:   src/roarm_main/moveit_servo/src/servo_parameters.cpp 	deleted:    src/roarm_main/moveit_servo/src/teleop_demo/joystick_servo_example (copy).cpp 	modified:   src/roarm_main/moveit_servo/src/teleop_demo/joystick_servo_example.cpp 	modified:   src/roarm_main/moveit_servo/test/servo_launch_test_common.hpp 	modified:   src/roarm_main/roarm_description/config/roarm_description.rviz 	deleted:    src/roarm_main/roarm_description/launch/gazebo.launch.py 	new file:   src/roarm_main/roarm_description/meshes/gripper_link.STL

File: src/roarm_main/roarm_description/urdf/roarm_description.urdf (robot description, URDF)
Before this commit: robot roarm_description, 5 links, 4 joints
Links:
- removed link link4
- added link gripper_link, mass 0.00365697683069397; collision mesh filename=package://roarm_description/meshes/gripper_link.STL; visual mesh filename=package://roarm_description/meshes/gripper_link.STL
- added link hand_tcp
Joints:
- removed joint link3_to_link4
- added joint link3_to_gripper_link: type revolute, parent link3, child gripper_link, origin xyz=0.002906 -0.21599 -0.00066683 rpy=-1.5708 0 -1.5708, axis 0 0 1, limit lower=0 upper=1.5 effort=0 velocity=0
- added joint link3_to_hand_tcp: type fixed, parent link3, child hand_tcp, origin xyz=0.002 -0.2802 0 rpy=-1.5708 0 -1.5708, axis 0 0 0
- joint base_link_to_link1: axis 0 0 1 -> 0 0 -1; limit lower=-3.1415926 upper=3.1415926 effort=0 velocity=0 -> lower=-3.1416 upper=3.1416 effort=0 velocity=0; origin xyz=0.01 0 0.0836 rpy=0 0 0 -> xyz=0.0100000008759151 0 0.123059270461044 rpy=0 0 0
- joint link1_to_link2: origin xyz=0 0.03618 0.039473 rpy=-1.5708 -1.5708 0 -> xyz=0 0 0 rpy=-1.5707963267949 -1.5707963267949 0
- joint link2_to_link3: limit lower=-1 upper=3.1415926 effort=0 velocity=0 -> lower=-1 upper=3.1416 effort=0 velocity=0; origin xyz=0.2368 0.030002 -0.01607 rpy=0 0 0 -> xyz=0.236815132922094 0.0300023995170449 0 rpy=0 0 1.5707963267949

File: src/roarm_main/roarm_description/urdf/roarm_description_web_app.urdf (robot description, URDF)
Before this commit: robot roarm_description, 5 links, 4 joints
Links:
- removed link link4
- added link gripper_link, mass 0.00365697683069397; collision mesh filename=package://roarm_description/meshes/gripper_link.STL; visual mesh filename=package://roarm_description/meshes/gripper_link.STL
- added link hand_tcp
Joints:
- removed joint link3_to_link4
- added joint link3_to_gripper_link: type revolute, parent link3, child gripper_link, origin xyz=0.002906 -0.21599 -0.00066683 rpy=-3.1415926 0 -1.5708, axis 0 0 1, limit lower=0 upper=1.5 effort=0 velocity=0
- added joint link3_to_hand_tcp: type fixed, parent link3, child hand_tcp, origin xyz=0.002 -0.2802 0 rpy=-1.5708 0 -1.5708, axis 0 0 0
- joint base_link_to_link1: axis 0 0 1 -> 0 0 -1; limit lower=-3.1415926 upper=3.1415926 effort=0 velocity=0 -> lower=-3.1416 upper=3.1416 effort=0 velocity=0; origin xyz=0.01 0 0.0836 rpy=0 0 0 -> xyz=0.0100000008759151 0 0.123059270461044 rpy=0 0 0
- joint link1_to_link2: origin xyz=0 0.03618 0.039473 rpy=-1.5708 -1.5708 0 -> xyz=0 0 0 rpy=-1.5707963267949 -1.5707963267949 0
- joint link2_to_link3: limit lower=-1 upper=3.1415926 effort=0 velocity=0 -> lower=-1 upper=3.1416 effort=0 velocity=0; origin xyz=0.2368 0.030002 -0.01607 rpy=0 0 0 -> xyz=0.236815132922094 0.0300023995170449 0 rpy=0 0 1.5707963267949

File: src/roarm_main/roarm_moveit/config/roarm_description.ros2_control.xacro (robot description, xacro)
@@ -29,8 +29,8 @@
                 <state_interface name="velocity"/>
             </joint>
-            <joint name="link3_to_link4">
+            <joint name="link3_to_gripper_link">
                 <command_interface name="position"/>
                 <state_interface name="position">
-                  <param name="initial_value">${initial_positions['link3_to_link4']}</param>
+                  <param name="initial_value">${initial_positions['link3_to_gripper_link']}</param>
                 </state_interface>
                 <state_interface name="velocity"/>
